Commit message: add joint_position_cmd to control the joints.

File: arm_typed_robot/urdf/arm_robot.urdf (robot description, URDF)
Before this commit: robot arm_robot, 6 links, 5 joints
Joints:
- removed joint elbow
- removed joint hip
- removed joint shoulder
- removed joint wrist
- added joint joint1: type continuous, parent base_link, child torso, origin xyz=0.0 0.0 0.05 rpy=0 0 1.5708, axis 0 0 1
- added joint joint2: type continuous, parent torso, child upper_arm, origin xyz=0.0 -0.1 0.45 rpy=0 1.5708 0, axis 0 1 0
- added joint joint3: type continuous, parent upper_arm, child lower_arm, origin xyz=0.0 0.1 0.35 rpy=0 0 0, axis 0 1 0
- added joint joint4: type continuous, parent lower_arm, child hand, origin xyz=0.0 0.0 0.425 rpy=0 0 0, axis 0 1 0
